File: hardware/magfest4.kicad_sch (KiCad schematic)
At the start: 38 parts, among them J1 AVR-ISP-6, J2 AVR-ISP-6, J3 USB_B_Micro, P1 CONN_1, P2 CONN_1, P3 CONN_1, P4 CONN_1, P5 CONN_1, P6 CONN_1, P7 CONN_1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

Commit message: Added LSCS parts
Parts:
- C1, C3, C4: LCSC (none) -> C13585
- C2: LCSC (none) -> C24497
- C5: LCSC (none) -> C90539
- C6, C7: LCSC (none) -> C577125
- C8, C9: LCSC (none) -> C97929
- D1: LCSC (none) -> C2980185
- D2: LCSC (none) -> C965822
- D3: LCSC (none) -> C130717
- J1, J2: LCSC (none) -> C65114
- J3: footprint Connector_USB:USB_Micro-B_Amphenol_10118193-0001LF_Horizontal -> magfest4:AMPHENOL_10118192-0001LF; LCSC (none) -> C132564
- P1, P2, P3, P4, P5, P6, P7, P8: now not fitted
- Q3: LCSC (none) -> C110474
- R1, R2: LCSC (none) -> C17927
- R10, R11: LCSC (none) -> C4410
- R3: LCSC (none) -> C25351
- R4, R6: LCSC (none) -> C2907384
- R5: LCSC (none) -> C26030
- R7, R8, R9: LCSC (none) -> C137240
- U1: footprint Package_SO:SOIC-8_3.9x4.9mm_P1.27mm -> Package_SO:SOIC-8_5.23x5.23mm_P1.27mm; LCSC (none) -> C1338203
- U2: LCSC (none) -> C412819
- X1: footprint Crystal:Crystal_SMD_1210-4Pin_1.2x1.0mm -> Crystal:Crystal_SMD_5032-2Pin_5.0x3.2mm; LCSC (none) -> C5182767

Commit message: Fix parts for JLCPCB
Parts:
- D1: LCSC C2980185 -> C434442
- U1: footprint Package_SO:SOIC-8_5.23x5.23mm_P1.27mm -> Package_SO:SOIC-8_3.9x4.9mm_P1.27mm
Changed lines of the file:
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@@
 			)
 		)
-		(property "Footprint" "Package_SO:SOIC-8_5.23x5.23mm_P1.27mm"
+		(property "Footprint" "Package_SO:SOIC-8_3.9x4.9mm_P1.27mm"
 			(at 72.39 49.53 0)
 			(effects
@@
 			)
 		)
-		(property "LCSC" "C2980185"
+		(property "LCSC" "C434442"
 			(at 224.79 140.97 0)
 			(effects
